File: hardware/bessy-c/bessy-c.kicad_sch (KiCad schematic)
At the start: 55 parts, among them J1 rotary_encoder, J10 fan, J11 auger, J2 probe0, J3 probe1, J4 probe2, J5 PTD, J6 igniter, J7 Display, J8 fire_pit, J9 line_in, K1 1462042-7, K2 1462042-7, K3 1462042-7, Q1 BC847, Q2 SCS-1002K, Q3 BC847, Q4 BC847, U1 ProS3, U2 ADS1115IDGS, U3 MCP96xx01x-x-MX, U4 IRM-10-5, U5 NAU7802SGI

Commit message: Ordered bessy-c pcba rev 1
Parts:
- removed K2, K3: 1462042-7, Digikey_1462042_7_Relay:IM-C_THRU_TEC, symbol Digikey_1462042_7_Relay:1462042-7
- removed Q2: SCS-1002K, Digikey_SCS_1002K:TRAN_SCS-1002K_SIG, symbol Digikey_SCS_1002K:SCS-1002K
- added C8: 10uF, Capacitor_SMD:C_0805_2012Metric, symbol Device:C
- added D1, D2, D3: 1N4148W, Diode_SMD:D_SOD-123, symbol Diode:1N4148W
- added D4: BZT52C24, Diode_SMD:D_SOD-123F, symbol Diode:BZT52Bxx
- added K2, K3: G5NB, Relay_THT:Relay_SPST_Omron_G5NB, symbol Relay:G5NB
- added R22: 10k, Resistor_SMD:R_0805_2012Metric, symbol Device:R
- added T1: ZMCT102, kicad-jcl-lib:XFMR_ZMCT102, symbol jcl-sym-lib:ZMCT102
- added U6: ADS1115IDGS, Package_SO:TSSOP-10_3x3mm_P0.5mm, symbol Analog_ADC:ADS1115IDGS
- C1, C2: symbol jcl-sym-lib:opl-C-0805-100nf -> Device:C; Link zoocode.dev -> (none); MPN CL21B102KDCNFNC -> (none)
- C3: symbol jcl-sym-lib:opl-C-0805-10uf -> Device:C; Link zoocode.dev -> (none); MPN CC0805KRX5R7BB106 -> (none)
- C4: symbol jcl-sym-lib:opl-C-0805-1uf -> Device:C; Link zoocode.dev -> (none); MPN CL21B105KLFVPNE -> (none)
- C5, C6, C7: value .1uF -> 0.1uF; symbol jcl-sym-lib:opl-C-0805-100nf -> Device:C; Link zoocode.dev -> (none); MPN CL21B102KDCNFNC -> (none)
- H1, H2, H3, H4: now not fitted
- J1: value rotary_encoder -> Conn_01x05; footprint TerminalBlock:TerminalBlock_MaiXu_MX126-5.0-05P_1x05_P5.00mm -> Connector_PinHeader_2.54mm:PinHeader_1x05_P2.54mm_Vertical; symbol Connector:Screw_Terminal_01x05 -> Connector_Generic:Conn_01x05; Label (none) -> encoder
- J10: value fan -> DB300V-5.0-2P-BK-S; Label (none) -> fan; now in the parts list
- J11: value auger -> DB300V-5.0-2P-BK-S; Label (none) -> auger; now in the parts list
- J2: value probe0 -> DB300V-5.0-2P-BK-S; Label (none) -> probe1; now in the parts list
- J3: value probe1 -> DB300V-5.0-2P-BK-S; Label (none) -> probe2; now in the parts list
- J4: value probe2 -> DB300V-5.0-2P-BK-S; Label (none) -> probe3; now in the parts list
- J5: value PTD -> DB300V-5.0-2P-BK-S; Label (none) -> chamber; now in the parts list
- J6: value igniter -> DB300V-5.0-2P-BK-S; Label (none) -> igniter; now in the parts list
- J7: value Display -> Conn_01x14; footprint Connector_PinHeader_2.54mm:PinHeader_1x15_P2.54mm_Vertical -> Connector_PinHeader_2.54mm:PinHeader_1x14_P2.54mm_Vertical; Label (none) -> display
- J8: value fire_pit -> DB300V-5.0-2P-BK-S; Label (none) -> firepot; now in the parts list
- J9: value line_in -> DB300V-5.0-2P-BK-S; Label (none) -> line_in; now in the parts list
- K1: value 1462042-7 -> G5NB; footprint Digikey_1462042_7_Relay:IM-C_THRU_TEC -> Relay_THT:Relay_SPST_Omron_G5NB; symbol Digikey_1462042_7_Relay:1462042-7 -> Relay:G5NB; now in the parts list
- Q1, Q3, Q4: value BC847 -> MMBT2222A; symbol jcl-sym-lib:opl-BC847 -> Transistor_BJT:MMBT2222A; Link https://www.seeedstudio.com/opl.html -> (none); MPN BC847B -> (none)
- R1, R10, R2, R20, R21: symbol jcl-sym-lib:opl-R-0805-100 -> Device:R; Link https://www.seeedstudio.com/opl.html -> (none); MPN CRCW0805100RFKEB -> (none)
- R11, R13, R15, R16, R3, R8: symbol jcl-sym-lib:opl-R-0805-4.7k -> Device:R; Link https://www.seeedstudio.com/opl.html -> (none); MPN 0805W8F4701T5E -> (none)
- R12, R14, R7, R9: symbol jcl-sym-lib:opl-R-0805-10k -> Device:R; Link https://www.seeedstudio.com/opl.html -> (none); MPN RC0805JR-0710KL -> (none)
- R17, R18: symbol jcl-sym-lib:opl-R-0805-47 -> Device:R; Link https://www.seeedstudio.com/opl.html -> (none); MPN ESR10EZPJ470 -> (none)
- R19: symbol jcl-sym-lib:opl-R-0805-3.3k -> Device:R; Link https://www.seeedstudio.com/opl.html -> (none); MPN RC0805JR-073K3L -> (none)
- R4, R5, R6: symbol jcl-sym-lib:opl-R-0805-47k -> Device:R; Link https://www.seeedstudio.com/opl.html -> (none); MPN 0805W8F4702T5E -> (none)
- U2: symbol jcl-sym-lib:opl-ADS1015IDGS -> Analog_ADC:ADS1115IDGS; Link https://www.seeedstudio.com/opl.html -> (none); MPN ADS1015IDGSR -> (none)
- U3: value MCP96xx01x-x-MX -> MCP96L00T-E/MX; symbol jcl-sym-lib:opl-MCP96xx01x-x-MX -> Sensor_Temperature:MCP96xx01x-x-MX; Link https://www.seeedstudio.com/opl.html -> (none); MPN MCP96L00T-E/MX -> (none)
- U4: now in the parts list
- U5: footprint SOI16_NAU7802SGI_NUV -> Digikey_NAU7802SGI:SOI16_NAU7802SGI_NUV; MPN NAU7802SGI -> (none)
Connections:
- net IO38 is gone; now on net tft_rst: U1.22 (IO38)
- net IO42 is gone; now on net auger: U1.18 (IO42)
- net IO44 is gone; now on net tft_dc: U1.23 (RX)
- net +3.3V: now also C8.1, R22.2, U6.8 (VDD)
- net +5V: now also K1.A1, D2.1 (K), D3.1 (K), D4.2 (A), K2.A1, K3.A1; no longer K1.8
- net GND: now also C8.2, U6.3 (GND); no longer R10.1
- net ac_a1: now also K3.14
- net ac_f1: now also K2.14
- net ac_i2: now also K1.14; no longer K1.5
- net ac_n: now also K1.13, K2.13, K3.13
- net auger: no longer U1.19 (IO41)
- net fan: now also U1.19 (IO41); no longer U1.20 (IO40)
- net i2c_scl: now also U6.10 (SCL)
- net i2c_sda: now also U6.9 (SDA)
- net igniter: now also U1.20 (IO40); no longer U1.21 (IO39)
- net tft_cs: now also U1.21 (IO39); no longer U1.16 (IO13)
- net tft_dc: no longer U1.17 (IO12)
- net at Q1.3 (C): now also K1.A2, D3.2 (A); no longer K1.1
- net at Q4.3 (C): now also D1.2 (A), K3.A2
- net at Q3.3 (C): now also D2.2 (A), K2.A2
- removed net ac_i1: K1.3
- removed net ac_i3: K1.7
- net igniter_current: no longer names the net of R10.2
- net igniter_current: now also T1.1, U6.6 (AIN2); no longer U2.7 (AIN3)
- new net: D1.1 (K), D4.1 (K)
- new net: R10.1, T1.2, U6.7 (AIN3)
- new net: R22.1, U6.1 (ADDR), U6.2 (ALERT/RDY)
- no-connect marks 36 -> 28
Other:
- company: (none) -> ${DESIGNER}
- title: (none) -> ${BOARD_NAME}
- moved on the sheet: C1, C2, C3, C4, C5, C6, C7, J10, J11, J2, J3, J4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

Commit message: r2 of board with bodge wires fixed
Parts:
- added C9: 0.1uF, Capacitor_SMD:C_0805_2012Metric, symbol Device:C
- T1: footprint kicad-jcl-lib:XFMR_ZMCT102 -> DigiKey-jcl:XFMR_ZMCT102; symbol jcl-sym-lib:ZMCT102 -> Digikey_jcl:ZMCT102
- U1: footprint kicad-jcl-lib:ProS3_SMD -> DigiKey-jcl:ProS3_SMD; symbol jcl-sym-lib:ProS3 -> Digikey_jcl:ProS3; now in the parts list
- U4: footprint Digikey_IRM_10_5:IRM-10_MWU -> DigiKey-jcl:IRM-10_MWU; symbol Digikey_IRM_10_5:IRM-10-5 -> Digikey_jcl:IRM-10-5
- U5: footprint Digikey_NAU7802SGI:SOI16_NAU7802SGI_NUV -> DigiKey-jcl:SOI16_NAU7802SGI_NUV; symbol Digikey_NAU7802SGI:NAU7802SGI -> Digikey_jcl:NAU7802SGI
Connections:
- net IO35 is gone; now on net ctc_int: U1.34 (IO35)
- net IO37 is gone; now on net ctc_rst: U1.33 (IO37)
- net GND: now also J5.2 (Pin_2), R17.2
- net at U5.4 (VIN2N): now also C9.2
- net at U5.5 (VIN2P): now also C9.1
- no-connect marks 28 -> 24
Other:
- moved on the sheet: J5
